Commit message: WORKING basic structure of launch and urdf files

File: src/rover_description/urdf/rover_s1.urdf.xacro (robot description, xacro)
@@ -1,5 +1,13 @@
 <?xml version="1.0"?>
-<robot name="rover_s1" xmlns:xacro="http://www.ros.org/wiki/xacro">
+<robot name="rover_s1" xmlns:xacro="http://playerstage.sourceforge.net/gazebo/xmlschema/#xacro">
+  <xacro:arg name="name" default=""/>
+  <xacro:property name="_name" value="$(arg name)"/>
+  <xacro:if value="${_name != ''}">
+    <xacro:property name="tf_prefix" value="${_name}/"/>
+  </xacro:if>
+  <xacro:if value="${_name == ''}">
+    <xacro:property name="tf_prefix" value=""/>
+  </xacro:if>
   <xacro:include filename="$(find rover_description)/urdf/suspension.urdf.xacro"/>
-  <xacro:suspension tf_prefix=""/>
+  <xacro:suspension tf_prefix="${tf_prefix}"/>
 </robot>

File: src/rover_description/urdf/suspension.urdf.xacro (robot description, xacro)
@@ -1,6 +1,7 @@
 <?xml version="1.0"?>
-<robot name="rover_s1" xmlns:xacro="http://www.ros.org/wiki/xacro">
+<robot name="rover_s1" xmlns:xacro="http://playerstage.sourceforge.net/gazebo/xmlschema/#xacro">
   <xacro:macro name="suspension" params="tf_prefix=''">
-    <link name="${tf_prefix}base_link">
+    <link name="${tf_prefix}base_link"/>
+    <link name="${tf_prefix}suspension_base_link">
       <inertial>
         <origin xyz="0 0 0.05" rpy="0 0 0"/>
@@ -11,22 +12,13 @@
         <origin xyz="0 0 0.05"/>
         <geometry>
-          <mesh filename="package://rover_description/meshes/suspension/central-axii.stl"/>
+          <mesh filename="package://rover_description/meshes/suspension/central-axii.stl" scale="0.01 0.01 0.01"/>
         </geometry>
       </visual>
-      <collision>
-        <origin xyz="0 0 0.05"/>
-        <geometry>
-          <mesh filename="package://rover_description/meshes/suspension/central-axii.stl"/>
-        </geometry>
-      </collision>
     </link>
+    <joint name="${tf_prefix}suspension_base_joint" type="fixed">
+      <origin xyz="0 0 0.03465" rpy="0 0 0"/>
+      <parent link="${tf_prefix}base_link"/>
+      <child link="${tf_prefix}suspension_base_link"/>
+    </joint>
   </xacro:macro>
-  <!-- Instantiate the suspension macro -->
-  <xacro:suspension tf_prefix=""/>
-  <joint name="fixed" type="fixed">
-    <parent link="world"/>
-    <child link="base_link"/>
-    <origin xyz="0 0 0" rpy="0 0 0"/>
-  </joint>
-  <link name="world"/>
 </robot>

Commit message: feat(suspension): Complete URDF configuration and RViz visualization

File: src/rover_description/urdf/rover_s1.urdf.xacro (robot description, xacro)
@@ -10,4 +10,12 @@
   </xacro:if>
   <xacro:include filename="$(find rover_description)/urdf/suspension.urdf.xacro"/>
-  <xacro:suspension tf_prefix="${tf_prefix}"/>
+  <xacro:include filename="$(find rover_description)/urdf/rocker.urdf.xacro"/>
+  <xacro:include filename="$(find rover_description)/urdf/wheel.urdf.xacro"/>
+  <xacro:suspension xyz="0 0 0" tf_prefix="${tf_prefix}"/>
+  <xacro:rocker name="left"  xyz="0 0.305 0"  side="1"  base_axii="suspension_base_link" tf_prefix="${tf_prefix}"/>
+  <xacro:rocker name="right" xyz="0 -0.305 0" side="-1" base_axii="suspension_base_link" tf_prefix="${tf_prefix}"/>
+  <xacro:wheel name="front_left"  x="0.53" y="0" z="0" side="1" base_rocker="left" tf_prefix="${tf_prefix}"/>
+  <xacro:wheel name="front_right" x="0.53" y="0" z="0" side="-1" base_rocker="right" tf_prefix="${tf_prefix}"/>
+  <xacro:wheel name="back_left"  x="-0.53" y="0" z="0" side="1"  base_rocker="left" tf_prefix="${tf_prefix}"/>
+  <xacro:wheel name="back_right" x="-0.53" y="0" z="0" side="-1" base_rocker="right" tf_prefix="${tf_prefix}"/>
 </robot>

File: src/rover_description/urdf/suspension.urdf.xacro (robot description, xacro)
@@ -1,24 +1,54 @@
 <?xml version="1.0"?>
 <robot name="rover_s1" xmlns:xacro="http://playerstage.sourceforge.net/gazebo/xmlschema/#xacro">
-  <xacro:macro name="suspension" params="tf_prefix=''">
+  <xacro:macro name="suspension" params="xyz tf_prefix=''">
     <link name="${tf_prefix}base_link"/>
     <link name="${tf_prefix}suspension_base_link">
       <inertial>
-        <origin xyz="0 0 0.05" rpy="0 0 0"/>
-        <mass value="10.0"/>
+        <origin xyz="0 0 0" rpy="0 0 0"/>
+        <mass value="0.5"/>
         <inertia ixx="0.5" ixy="0" ixz="0" iyy="0.5" iyz="0" izz="1.0"/>
       </inertial>
       <visual>
-        <origin xyz="0 0 0.05"/>
+        <origin xyz="0 -0.325 0"/>
         <geometry>
-          <mesh filename="package://rover_description/meshes/suspension/central-axii.stl" scale="0.01 0.01 0.01"/>
+          <mesh filename="package://rover_description/meshes/suspension/central_axii.stl" scale="0.001 0.001 0.001"/>
         </geometry>
       </visual>
     </link>
     <joint name="${tf_prefix}suspension_base_joint" type="fixed">
-      <origin xyz="0 0 0.03465" rpy="0 0 0"/>
+      <origin xyz="${xyz}" rpy="0 0 0"/>
       <parent link="${tf_prefix}base_link"/>
       <child link="${tf_prefix}suspension_base_link"/>
     </joint>
   </xacro:macro>
+    <material name="armor_plastic">
+      <color rgba="0.2277128 0.2277128 0.2277128 0.8"/>
+    </material>
+    <material name="chassis">
+      <color rgba="0.0981132 0.0981132 0.0981132 1.0"/>
+    </material>
+    <material name="cover_plastic">
+      <color rgba="0.2548322 0.2548322 0.2548322 0.30000000000000004"/>
+    </material>
+    <material name="dark_plastic">
+      <color rgba="0.0281746 0.0281746 0.0281746 1.0"/>
+    </material>
+    <material name="metal">
+      <color rgba="0.0281746 0.028 0.0281746 1.0"/>
+    </material>
+    <material name="hit_detector">
+      <color rgba="0.1697846 0.1697846 0.1697846 1.0"/>
+    </material>
+    <material name="led_light">
+      <color rgba="0 0.7773585 0.7773583 1.0"/>
+    </material>
+    <material name="wheel_plastic">
+      <color rgba="0.2739087 0.2739087 0.2739087 1.0"/>
+    </material>
+    <material name="EP_up.001">
+      <color rgba="0.0284811 0.0284811 0.0284811 1.0"/>
+    </material>
+    <material name="steel">
+      <color rgba="0.675 0.69453125 0.69453125 1.0"/>
+    </material>
 </robot>
