Commit message: Fix wheel position

File: src/indomitus_rover_description/urdf/wheel.urdf.xacro (robot description, xacro)
@@ -47,5 +47,5 @@
     </link>
     <joint name="${tf_prefix}${name}_wheel_joint" type="continuous">
-      <origin xyz="0 0 -0.25" rpy="0 0 0"/>
+      <origin xyz="0 0 -0.27" rpy="0 0 0"/>
       <parent link="${tf_prefix}${name}_wheel_mount_link"/>
       <child link="${tf_prefix}${name}_wheel_link"/>
