Commit message: Fix control via teleop_twist

File: src/indomitus_rover_description/urdf/rocker.urdf.xacro (robot description, xacro)
@@ -30,5 +30,6 @@
       <child link="${tf_prefix}${name}_rocker_link"/>
       <axis xyz="0 1.0 0"/>
-      <limit effort="0" velocity="0"/>
+      <limit effort="100" velocity="1.0"/>
+      <dynamics damping="0.5" friction="0.1"/>
     </joint>
   </xacro:macro>

File: src/indomitus_rover_description/urdf/wheel.urdf.xacro (robot description, xacro)
@@ -21,5 +21,5 @@
       <child link="${tf_prefix}${name}_wheel_mount_link"/>
       <axis xyz="0 0 1"/>  <!-- вертикальна вісь (Z) для steering -->
-      <limit lower="${-pi/4}" upper="${pi/3}" effort="10" velocity="1"/>
+      <limit lower="${-pi/2}" upper="${pi/2}" effort="10" velocity="1"/>
     </joint>
     <link name="${tf_prefix}${name}_wheel_link">

Commit message: Add dependencies for rviz2; Add collisions for wheel_mount and rocker

File: src/indomitus_rover_description/urdf/rocker.urdf.xacro (robot description, xacro)
@@ -15,13 +15,11 @@
         <material name="steel"/>
       </visual>
-      <!-- <collision name="${name}_wheel">
-        <origin xyz="0 0 0" rpy="${pi/2} 0 0"/>
+      <collision>
+        <origin xyz="0 0 0" rpy="0 0 0"/>
+        <!-- <origin xyz="-0.55 ${0.02 * side} -0.04" rpy="0 0 0"/> -->
         <geometry>
-          <cylinder radius="0.05" length="0.042"/>
+          <box size="1.1 ${0.04 * side} 0.08"/> <!-- приблизно вдвічі масштаб visual -->
         </geometry>
-        <material name="collision">
-          <color rgba="0.8 0.0 0.0 1.0"/>
-        </material>
-      </collision> -->
+      </collision>
     </link>
     <joint name="${tf_prefix}${name}_rocker_joint" type="continuous">

File: src/indomitus_rover_description/urdf/wheel.urdf.xacro (robot description, xacro)
@@ -15,4 +15,10 @@
         <material name="steel"/>
       </visual>
+      <collision>
+        <origin xyz="0 ${0.11125 * side} -0.18" rpy="0 0 0" />
+        <geometry>
+          <box size="0.07 0.0625 0.25"/>
+        </geometry>
+      </collision>
     </link>
     <joint name="${tf_prefix}${name}_wheel_mount_joint" type="revolute">

Commit message: Temporary remove collision for rocker, FIX required, what is problem

File: src/indomitus_rover_description/urdf/rocker.urdf.xacro (robot description, xacro)
@@ -15,11 +15,4 @@
         <material name="steel"/>
       </visual>
-      <collision>
-        <origin xyz="0 0 0" rpy="0 0 0"/>
-        <!-- <origin xyz="-0.55 ${0.02 * side} -0.04" rpy="0 0 0"/> -->
-        <geometry>
-          <box size="1.1 ${0.04 * side} 0.08"/> <!-- приблизно вдвічі масштаб visual -->
-        </geometry>
-      </collision>
     </link>
     <joint name="${tf_prefix}${name}_rocker_joint" type="continuous">
