Commit message: Attached camera to camera_link in bridge_parameters

File: src/indomitus_rover_description/urdf/camera.urdf.xacro (robot description, xacro)
@@ -1,5 +1,5 @@
 <?xml version="1.0"?>
 <robot xmlns:xacro="https://www.ros.org/wiki/xacro">
-  <xacro:macro name="camera" params="tf_prefix:='' parent_link:='base_link'">
+  <xacro:macro name="camera" params="tf_prefix:='' parent_link:='main_body_link'">
     <link name="${tf_prefix}camera_link">
       <inertial>
@@ -27,5 +27,5 @@
       <parent link="${tf_prefix}${parent_link}"/>
       <child link="${tf_prefix}camera_link"/>
-      <origin xyz="0.3 0 0.6" rpy="0 0 0"/>
+      <origin xyz="0.3 0 0.1" rpy="0 0 0"/>
     </joint>
     <gazebo reference="${tf_prefix}camera_link">

File: src/indomitus_rover_description/urdf/indomitus_rover_s1.urdf.xacro (robot description, xacro)
@@ -1,4 +1,4 @@
 <?xml version="1.0"?>
-<robot name="indomitus_s1">
+<robot name="indomitus_s1" xmlns:xacro="http://www.ros.org/wiki/xacro">
   <!-- ===================== MATERIALS ===================== -->
   <material name="blue_body">
@@ -71,12 +71,15 @@
     </collision>
   </link>
-  <joint name="main_body_joint" type="revolute">
+  <joint name="main_body_joint" type="fixed">
     <parent link="suspension_base_axii_link"/>
     <child link="main_body_link"/>
     <origin xyz="-0.04 0 0.05" rpy="0 0 0"/>
-    <axis xyz="0 1 0"/>
-    <limit lower="-1.0" upper="1.0" effort="10000" velocity="5.0"/>
-    <dynamics damping="20.0" friction="1.0"/>
-  </joint>
+    <!-- <axis xyz="0 1 0"/> -->
+    <!-- <limit lower="-1.0" upper="1.0" effort="10000" velocity="5.0"/> -->
+    <!-- <dynamics damping="20.0" friction="1.0"/> -->
+  </joint>
+  <!-- ===================== CAMERA ===================== -->
+  <xacro:include filename="$(find indomitus_rover_description)/urdf/camera.urdf.xacro"/>
+  <xacro:camera/>
   <!-- ===================== LEFT ROCKER ===================== -->
   <link name="l_rocker_link">

Commit message: Fix camera topic names, rqt output; fix license copyrights

File: src/indomitus_rover_description/urdf/camera.urdf.xacro (robot description, xacro)
@@ -30,20 +30,21 @@
     </joint>
     <gazebo reference="${tf_prefix}camera_link">
-    <sensor name="${tf_prefix}camera_rgb" type="camera">
-        <always_on>true</always_on>
-        <update_rate>30</update_rate>
-        <camera>
-        <horizontal_fov>1.396</horizontal_fov>
-        <image>
-            <width>640</width>
-            <height>480</height>
-            <format>R8G8B8</format>
-        </image>
-        <clip>
-            <near>0.1</near>
-            <far>100.0</far>
-        </clip>
-        </camera>
-    </sensor>
+      <sensor name="${tf_prefix}camera_rgb" type="camera">
+          <always_on>true</always_on>
+          <update_rate>30</update_rate>
+          <topic>camera/front_rgb/image_raw</topic>
+          <camera>
+            <horizontal_fov>1.396</horizontal_fov>
+            <image>
+                <width>640</width>
+                <height>480</height>
+                <format>R8G8B8</format>
+            </image>
+            <clip>
+                <near>0.1</near>
+                <far>100.0</far>
+            </clip>
+          </camera>
+      </sensor>
     </gazebo>
   </xacro:macro>

File: src/indomitus_rover_description/urdf/indomitus_rover_s1.urdf.xacro (robot description, xacro)
@@ -75,7 +75,4 @@
     <child link="main_body_link"/>
     <origin xyz="-0.04 0 0.05" rpy="0 0 0"/>
-    <!-- <axis xyz="0 1 0"/> -->
-    <!-- <limit lower="-1.0" upper="1.0" effort="10000" velocity="5.0"/> -->
-    <!-- <dynamics damping="20.0" friction="1.0"/> -->
   </joint>
   <!-- ===================== CAMERA ===================== -->
@@ -369,25 +366,2 @@
   </joint>
 </robot>
-<!-- <?xml version="1.0"?>
-<robot name="indomitus_s1" xmlns:xacro="https://www.ros.org/wiki/xacro">
-  <xacro:arg name="name" default=""/>
-  <xacro:property name="_name" value="$(arg name)"/>
-  <xacro:if value="${_name != ''}">
-    <xacro:property name="tf_prefix" value="${_name}/"/>
-  </xacro:if>
-  <xacro:if value="${_name == ''}">
-    <xacro:property name="tf_prefix" value=""/>
-  </xacro:if>
-  <xacro:include filename="$(find indomitus_rover_description)/urdf/suspension.urdf.xacro"/>
-  <xacro:include filename="$(find indomitus_rover_description)/urdf/rocker.urdf.xacro"/>
-  <xacro:include filename="$(find indomitus_rover_description)/urdf/wheel.urdf.xacro"/>
-  <xacro:include filename="$(find indomitus_rover_description)/urdf/camera.urdf.xacro"/>
-  <xacro:camera tf_prefix="${tf_prefix}"/>
-  <xacro:suspension xyz="0 0 0.4" tf_prefix="${tf_prefix}"/>
-  <xacro:rocker name="l"  xyz="0 0.305 0"  side="1"  base_axii="suspension_base_axii_link" tf_prefix="${tf_prefix}"/>
-  <xacro:rocker name="r" xyz="0 -0.305 0" side="-1" base_axii="suspension_base_axii_link" tf_prefix="${tf_prefix}"/>
-  <xacro:wheel name="fl"  x="0.53" y="0" z="0" side="1" base_rocker="l" tf_prefix="${tf_prefix}"/>
-  <xacro:wheel name="fr" x="0.53" y="0" z="0" side="-1" base_rocker="r" tf_prefix="${tf_prefix}"/>
-  <xacro:wheel name="bl"  x="-0.53" y="0" z="0" side="1"  base_rocker="l" tf_prefix="${tf_prefix}"/>
-  <xacro:wheel name="br" x="-0.53" y="0" z="0" side="-1" base_rocker="r" tf_prefix="${tf_prefix}"/>
-</robot> -->
