Commit message: Rename packages names to new rover name indomitus_rover

File: src/indomitus_rover_description/urdf/indomitus_rover_s1.urdf.xacro (robot description, xacro)
@@ -1,4 +1,4 @@
 <?xml version="1.0"?>
-<robot name="rover_s1" xmlns:xacro="http://playerstage.sourceforge.net/gazebo/xmlschema/#xacro">
+<robot name="indomitus_s1" xmlns:xacro="http://playerstage.sourceforge.net/gazebo/xmlschema/#xacro">
   <xacro:arg name="name" default=""/>
   <xacro:property name="_name" value="$(arg name)"/>
@@ -9,7 +9,7 @@
     <xacro:property name="tf_prefix" value=""/>
   </xacro:if>
-  <xacro:include filename="$(find rover_description)/urdf/suspension.urdf.xacro"/>
-  <xacro:include filename="$(find rover_description)/urdf/rocker.urdf.xacro"/>
-  <xacro:include filename="$(find rover_description)/urdf/wheel.urdf.xacro"/>
+  <xacro:include filename="$(find indomitus_rover_description)/urdf/suspension.urdf.xacro"/>
+  <xacro:include filename="$(find indomitus_rover_description)/urdf/rocker.urdf.xacro"/>
+  <xacro:include filename="$(find indomitus_rover_description)/urdf/wheel.urdf.xacro"/>
   <xacro:suspension xyz="0 0 0" tf_prefix="${tf_prefix}"/>
   <xacro:rocker name="left"  xyz="0 0.305 0"  side="1"  base_axii="suspension_base_link" tf_prefix="${tf_prefix}"/>

File: src/indomitus_rover_description/urdf/rocker.urdf.xacro (robot description, xacro)
@@ -11,5 +11,5 @@
         <origin xyz="-0.55 ${0.02 * side} -0.04" rpy="0 0 0"/>
         <geometry>
-          <mesh filename="package://rover_description/meshes/suspension/rocker.stl" scale="0.001 ${0.001 * side} 0.001"/>
+          <mesh filename="package://indomitus_rover_description/meshes/suspension/rocker.stl" scale="0.001 ${0.001 * side} 0.001"/>
         </geometry>
         <material name="steel"/>

File: src/indomitus_rover_description/urdf/suspension.urdf.xacro (robot description, xacro)
@@ -12,5 +12,5 @@
         <origin xyz="0 -0.325 0"/>
         <geometry>
-          <mesh filename="package://rover_description/meshes/suspension/central_axii.stl" scale="0.001 0.001 0.001"/>
+          <mesh filename="package://indomitus_rover_description/meshes/suspension/central_axii.stl" scale="0.001 0.001 0.001"/>
         </geometry>
       </visual>

File: src/indomitus_rover_description/urdf/wheel.urdf.xacro (robot description, xacro)
@@ -11,5 +11,5 @@
         <origin xyz="0 ${-0.06 * side} -0.269" rpy="0 0 0"/>
         <geometry>
-          <mesh filename="package://rover_description/meshes/suspension/wheel_mount.stl" scale="0.001 ${0.001 * side} 0.001"/>
+          <mesh filename="package://indomitus_rover_description/meshes/suspension/wheel_mount.stl" scale="0.001 ${0.001 * side} 0.001"/>
         </geometry>
         <material name="steel"/>
@@ -27,5 +27,5 @@
         <origin xyz="0 ${-0.06 * side} 0" rpy="${-pi/2} 0 0"/> <!-- ${0.12 * side} -->
         <geometry>
-          <mesh filename="package://rover_description/meshes/suspension/wheel.stl" scale="0.001 0.001 ${side * 0.001}"/>
+          <mesh filename="package://indomitus_rover_description/meshes/suspension/wheel.stl" scale="0.001 0.001 ${side * 0.001}"/>
         </geometry>
         <material name="wheel_plastic"/>

Commit message: First working version; add gazebo launch files; add inertia to wheels; Add gazebo-ros2 topics bridge

File: src/indomitus_rover_description/urdf/indomitus_rover_s1.urdf.xacro (robot description, xacro)
@@ -12,5 +12,5 @@
   <xacro:include filename="$(find indomitus_rover_description)/urdf/rocker.urdf.xacro"/>
   <xacro:include filename="$(find indomitus_rover_description)/urdf/wheel.urdf.xacro"/>
-  <xacro:suspension xyz="0 0 0" tf_prefix="${tf_prefix}"/>
+  <xacro:suspension xyz="0 0 0.4" tf_prefix="${tf_prefix}"/>
   <xacro:rocker name="left"  xyz="0 0.305 0"  side="1"  base_axii="suspension_base_link" tf_prefix="${tf_prefix}"/>
   <xacro:rocker name="right" xyz="0 -0.305 0" side="-1" base_axii="suspension_base_link" tf_prefix="${tf_prefix}"/>

File: src/indomitus_rover_description/urdf/wheel.urdf.xacro (robot description, xacro)
@@ -24,4 +24,11 @@
     </joint>
     <link name="${tf_prefix}${name}_wheel_link">
+      <inertial>
+        <origin xyz="0 0 0" rpy="0 0 0"/>
+        <mass value="0.5"/>
+        <inertia ixx="0.00563" ixy="0" ixz="0"
+                iyy="0.00563" iyz="0"
+                izz="0.01125"/>
+      </inertial>
       <visual>
         <origin xyz="0 ${-0.06 * side} 0" rpy="${-pi/2} 0 0"/> <!-- ${0.12 * side} -->

Commit message: Add sdf files and scripts for gz with sdf; rename launch files

File: src/indomitus_rover_description/urdf/indomitus_rover_s1.urdf.xacro (robot description, xacro)
@@ -15,6 +15,6 @@
   <xacro:camera tf_prefix="${tf_prefix}"/>
   <xacro:suspension xyz="0 0 0.4" tf_prefix="${tf_prefix}"/>
-  <xacro:rocker name="l"  xyz="0 0.305 0"  side="1"  base_axii="suspension_base_link" tf_prefix="${tf_prefix}"/>
-  <xacro:rocker name="r" xyz="0 -0.305 0" side="-1" base_axii="suspension_base_link" tf_prefix="${tf_prefix}"/>
+  <xacro:rocker name="l"  xyz="0 0.305 0"  side="1"  base_axii="suspension_base_axii_link" tf_prefix="${tf_prefix}"/>
+  <xacro:rocker name="r" xyz="0 -0.305 0" side="-1" base_axii="suspension_base_axii_link" tf_prefix="${tf_prefix}"/>
   <xacro:wheel name="fl"  x="0.53" y="0" z="0" side="1" base_rocker="l" tf_prefix="${tf_prefix}"/>
   <xacro:wheel name="fr" x="0.53" y="0" z="0" side="-1" base_rocker="r" tf_prefix="${tf_prefix}"/>

File: src/indomitus_rover_description/urdf/suspension.urdf.xacro (robot description, xacro)
@@ -3,5 +3,5 @@
   <xacro:macro name="suspension" params="xyz tf_prefix=''">
     <link name="${tf_prefix}base_link"/>
-    <link name="${tf_prefix}suspension_base_link">
+    <link name="${tf_prefix}suspension_base_axii_link">
       <inertial>
         <origin xyz="0 0 0" rpy="0 0 0"/>
@@ -16,8 +16,8 @@
       </visual>
     </link>
-    <joint name="${tf_prefix}suspension_base_joint" type="fixed">
+    <joint name="${tf_prefix}suspension_base_axii_joint" type="fixed">
       <origin xyz="${xyz}" rpy="0 0 0"/>
       <parent link="${tf_prefix}base_link"/>
-      <child link="${tf_prefix}suspension_base_link"/>
+      <child link="${tf_prefix}suspension_base_axii_link"/>
     </joint>
   </xacro:macro>

Commit message: Differential bar soft emulation with urdf model, working version

File: src/indomitus_rover_description/urdf/indomitus_rover_s1.urdf.xacro (robot description, xacro)
@@ -1,3 +1,370 @@
 <?xml version="1.0"?>
+<robot name="indomitus_s1">
+  <!-- ===================== MATERIALS ===================== -->
+  <material name="blue_body">
+    <color rgba="0.2 0.4 0.8 1"/>
+  </material>
+  <material name="grey_structure">
+    <color rgba="0.6 0.6 0.6 1"/>
+  </material>
+  <material name="orange_mount">
+    <color rgba="0.8 0.4 0.0 1"/>
+  </material>
+  <material name="dark_wheel">
+    <color rgba="0.1 0.1 0.1 1"/>
+  </material>
+  <material name="red_axii">
+    <color rgba="0.4 0.4 0.4 1"/>
+  </material>
+  <!-- ===================== BASE ===================== -->
+  <link name="base_link">
+    <inertial>
+      <mass value="0.1"/>
+      <inertia ixx="0.01" iyy="0.01" izz="0.01" ixy="0" ixz="0" iyz="0"/>
+    </inertial>
+  </link>
+  <!-- ===================== SUSPENSION BASE AXII ===================== -->
+  <link name="suspension_base_axii_link">
+    <inertial>
+      <origin xyz="0 0 0" rpy="0 0 0"/>
+      <mass value="0.5"/>
+      <inertia ixx="0.5" iyy="0.5" izz="1.0" ixy="0" ixz="0" iyz="0"/>
+    </inertial>
+    <visual>
+      <origin xyz="0 -0.325 0" rpy="0 0 0"/>
+      <geometry>
+        <mesh filename="package://indomitus_rover_description/meshes/suspension/central_axii.stl" scale="0.001 0.001 0.001"/>
+      </geometry>
+      <material name="red_axii"/>
+    </visual>
+    <collision>
+      <origin xyz="0 0 0" rpy="0 0 0"/>
+      <geometry>
+        <box size="0.1 0.65 0.05"/>
+      </geometry>
+    </collision>
+  </link>
+  <joint name="suspension_base_axii_joint" type="fixed">
+    <parent link="base_link"/>
+    <child link="suspension_base_axii_link"/>
+    <origin xyz="0 0 0" rpy="0 0 0"/>
+  </joint>
+  <!-- ===================== MAIN BODY ===================== -->
+  <link name="main_body_link">
+    <inertial>
+      <origin xyz="0 0 0" rpy="0 0 0"/>
+      <mass value="40.0"/>
+      <inertia ixx="0.608" iyy="1.283" izz="1.733" ixy="0" ixz="0" iyz="0"/>
+    </inertial>
+    <visual>
+      <origin xyz="0 0 0" rpy="0 0 0"/>
+      <geometry>
+        <box size="0.6 0.4 0.2"/>
+      </geometry>
+      <material name="blue_body"/>
+    </visual>
+    <collision>
+      <origin xyz="0 0 0" rpy="0 0 0"/>
+      <geometry>
+        <box size="0.6 0.4 0.15"/>
+      </geometry>
+    </collision>
+  </link>
+  <joint name="main_body_joint" type="revolute">
+    <parent link="suspension_base_axii_link"/>
+    <child link="main_body_link"/>
+    <origin xyz="-0.04 0 0.05" rpy="0 0 0"/>
+    <axis xyz="0 1 0"/>
+    <limit lower="-1.0" upper="1.0" effort="10000" velocity="5.0"/>
+    <dynamics damping="20.0" friction="1.0"/>
+  </joint>
+  <!-- ===================== LEFT ROCKER ===================== -->
+  <link name="l_rocker_link">
+    <inertial>
+      <origin xyz="0 0 0" rpy="0 0 0"/>
+      <mass value="1.0"/>
+      <inertia ixx="0.01" iyy="0.01" izz="0.01" ixy="0" ixz="0" iyz="0"/>
+    </inertial>
+    <visual>
+      <origin xyz="-0.55 0.02 -0.04" rpy="0 0 0"/>
+      <geometry>
+        <mesh filename="package://indomitus_rover_description/meshes/suspension/rocker.stl" scale="0.001 0.001 0.001"/>
+      </geometry>
+      <material name="grey_structure"/>
+    </visual>
+    <collision>
+      <origin xyz="0 0 0" rpy="0 0 0"/>
+      <geometry>
+        <box size="1.1 0.04 0.08"/>
+      </geometry>
+    </collision>
+  </link>
+  <joint name="l_rocker_joint" type="revolute">
+    <parent link="suspension_base_axii_link"/>
+    <child link="l_rocker_link"/>
+    <origin xyz="0 0.305 0" rpy="0 0 0"/>
+    <axis xyz="0 1 0"/>
+    <limit lower="-0.5" upper="0.5" effort="100" velocity="1.0"/>
+    <dynamics damping="0.5" friction="0.1"/>
+  </joint>
+  <!-- ===================== RIGHT ROCKER ===================== -->
+  <link name="r_rocker_link">
+    <inertial>
+      <origin xyz="0 0 0" rpy="0 0 0"/>
+      <mass value="1.0"/>
+      <inertia ixx="0.01" iyy="0.01" izz="0.01" ixy="0" ixz="0" iyz="0"/>
+    </inertial>
+    <visual>
+      <origin xyz="-0.55 0.02 -0.04" rpy="0 0 0"/>
+      <geometry>
+        <mesh filename="package://indomitus_rover_description/meshes/suspension/rocker.stl" scale="0.001 0.001 0.001"/>
+      </geometry>
+      <material name="grey_structure"/>
+    </visual>
+    <collision>
+      <origin xyz="0 0 0" rpy="0 0 0"/>
+      <geometry>
+        <box size="1.1 0.04 0.08"/>
+      </geometry>
+    </collision>
+  </link>
+  <joint name="r_rocker_joint" type="revolute">
+    <parent link="suspension_base_axii_link"/>
+    <child link="r_rocker_link"/>
+    <origin xyz="0 -0.305 0" rpy="0 0 0"/>
+    <axis xyz="0 1 0"/>
+    <limit lower="-0.5" upper="0.5" effort="100" velocity="1.0"/>
+    <dynamics damping="0.5" friction="0.1"/>
+  </joint>
+  <!-- ===================== FRONT LEFT WHEEL MOUNT ===================== -->
+  <link name="fl_wheel_mount_link">
+    <inertial>
+      <origin xyz="0 0 0" rpy="0 0 0"/>
+      <mass value="0.162"/>
+      <inertia ixx="0.0002" iyy="0.00012" izz="0.00012" ixy="0" ixz="0" iyz="0"/>
+    </inertial>
+    <visual>
+      <origin xyz="0 -0.06 -0.269" rpy="0 0 0"/>
+      <geometry>
+        <mesh filename="package://indomitus_rover_description/meshes/suspension/wheel_mount.stl" scale="0.001 0.001 0.001"/>
+      </geometry>
+      <material name="orange_mount"/>
+    </visual>
+    <collision>
+      <origin xyz="0 0.11125 -0.18" rpy="0 0 0"/>
+      <geometry>
+        <box size="0.07 0.0625 0.25"/>
+      </geometry>
+    </collision>
+  </link>
+  <joint name="fl_wheel_mount_joint" type="revolute">
+    <parent link="l_rocker_link"/>
+    <child link="fl_wheel_mount_link"/>
+    <origin xyz="0.53 0 0" rpy="0 0 0"/>
+    <axis xyz="0 0 1"/>
+    <limit lower="-1.5708" upper="1.5708" effort="500" velocity="2"/>
+    <dynamics damping="0.5" friction="0.3"/>
+  </joint>
+  <!-- ===================== FRONT LEFT WHEEL ===================== -->
+  <link name="fl_wheel_link">
+    <inertial>
+      <origin xyz="0 0 0" rpy="0 0 0"/>
+      <mass value="0.5"/>
+      <inertia ixx="0.00563" iyy="0.00563" izz="0.01125" ixy="0" ixz="0" iyz="0"/>
+    </inertial>
+    <visual>
+      <origin xyz="0 -0.06 0" rpy="-1.5708 0 0"/>
+      <geometry>
+        <mesh filename="package://indomitus_rover_description/meshes/suspension/wheel.stl" scale="0.001 0.001 0.001"/>
+      </geometry>
+      <material name="dark_wheel"/>
+    </visual>
+    <collision>
+      <origin xyz="0 0 0" rpy="1.5708 0 0"/>
+      <geometry>
+        <cylinder radius="0.15" length="0.12"/>
+      </geometry>
+    </collision>
+  </link>
+  <joint name="fl_wheel_joint" type="continuous">
+    <parent link="fl_wheel_mount_link"/>
+    <child link="fl_wheel_link"/>
+    <origin xyz="0 0 -0.27" rpy="0 0 0"/>
+    <axis xyz="0 1 0"/>
+    <limit effort="100" velocity="10"/>
+  </joint>
+  <!-- ===================== FRONT RIGHT WHEEL MOUNT ===================== -->
+  <link name="fr_wheel_mount_link">
+    <inertial>
+      <origin xyz="0 0 0" rpy="0 0 0"/>
+      <mass value="0.162"/>
+      <inertia ixx="0.0002" iyy="0.00012" izz="0.00012" ixy="0" ixz="0" iyz="0"/>
+    </inertial>
+    <visual>
+      <origin xyz="0 0.06 -0.269" rpy="0 0 3.14159"/>
+      <geometry>
+        <mesh filename="package://indomitus_rover_description/meshes/suspension/wheel_mount.stl" scale="0.001 0.001 0.001"/>
+      </geometry>
+      <material name="orange_mount"/>
+    </visual>
+    <collision>
+      <origin xyz="0 -0.11125 -0.18" rpy="0 0 0"/>
+      <geometry>
+        <box size="0.07 0.0625 0.25"/>
+      </geometry>
+    </collision>
+  </link>
+  <joint name="fr_wheel_mount_joint" type="revolute">
+    <parent link="r_rocker_link"/>
+    <child link="fr_wheel_mount_link"/>
+    <origin xyz="0.53 0 0" rpy="0 0 0"/>
+    <axis xyz="0 0 1"/>
+    <limit lower="-1.5708" upper="1.5708" effort="500" velocity="2"/>
+    <dynamics damping="0.5" friction="0.3"/>
+  </joint>
+  <!-- ===================== FRONT RIGHT WHEEL ===================== -->
+  <link name="fr_wheel_link">
+    <inertial>
+      <origin xyz="0 0 0" rpy="0 0 0"/>
+      <mass value="0.5"/>
+      <inertia ixx="0.00563" iyy="0.00563" izz="0.01125" ixy="0" ixz="0" iyz="0"/>
+    </inertial>
+    <visual>
+      <origin xyz="0 0.06 0" rpy="-1.5708 0 3.14159"/>
+      <geometry>
+        <mesh filename="package://indomitus_rover_description/meshes/suspension/wheel.stl" scale="0.001 0.001 0.001"/>
+      </geometry>
+      <material name="dark_wheel"/>
+    </visual>
+    <collision>
+      <origin xyz="0 0 0" rpy="-1.5708 0 0"/>
+      <geometry>
+        <cylinder radius="0.15" length="0.12"/>
+      </geometry>
+    </collision>
+  </link>
+  <joint name="fr_wheel_joint" type="continuous">
+    <parent link="fr_wheel_mount_link"/>
+    <child link="fr_wheel_link"/>
+    <origin xyz="0 0 -0.27" rpy="0 0 0"/>
+    <axis xyz="0 1 0"/>
+    <limit effort="100" velocity="10"/>
+  </joint>
+  <!-- ===================== BACK LEFT WHEEL MOUNT ===================== -->
+  <link name="bl_wheel_mount_link">
+    <inertial>
+      <origin xyz="0 0 0" rpy="0 0 0"/>
+      <mass value="0.162"/>
+      <inertia ixx="0.0002" iyy="0.00012" izz="0.00012" ixy="0" ixz="0" iyz="0"/>
+    </inertial>
+    <visual>
+      <origin xyz="0 -0.06 -0.269" rpy="0 0 0"/>
+      <geometry>
+        <mesh filename="package://indomitus_rover_description/meshes/suspension/wheel_mount.stl" scale="0.001 0.001 0.001"/>
+      </geometry>
+      <material name="orange_mount"/>
+    </visual>
+    <collision>
+      <origin xyz="0 0.11125 -0.18" rpy="0 0 0"/>
+      <geometry>
+        <box size="0.07 0.0625 0.25"/>
+      </geometry>
+    </collision>
+  </link>
+  <joint name="bl_wheel_mount_joint" type="revolute">
+    <parent link="l_rocker_link"/>
+    <child link="bl_wheel_mount_link"/>
+    <origin xyz="-0.53 0 0" rpy="0 0 0"/>
+    <axis xyz="0 0 1"/>
+    <limit lower="-1.5708" upper="1.5708" effort="500" velocity="2"/>
+    <dynamics damping="0.5" friction="0.3"/>
+  </joint>
+  <!-- ===================== BACK LEFT WHEEL ===================== -->
+  <link name="bl_wheel_link">
+    <inertial>
+      <origin xyz="0 0 0" rpy="0 0 0"/>
+      <mass value="0.5"/>
+      <inertia ixx="0.00563" iyy="0.00563" izz="0.01125" ixy="0" ixz="0" iyz="0"/>
+    </inertial>
+    <visual>
+      <origin xyz="0 -0.06 0" rpy="-1.5708 0 0"/>
+      <geometry>
+        <mesh filename="package://indomitus_rover_description/meshes/suspension/wheel.stl" scale="0.001 0.001 0.001"/>
+      </geometry>
+      <material name="dark_wheel"/>
+    </visual>
+    <collision>
+      <origin xyz="0 0 0" rpy="1.5708 0 0"/>
+      <geometry>
+        <cylinder radius="0.15" length="0.12"/>
+      </geometry>
+    </collision>
+  </link>
+  <joint name="bl_wheel_joint" type="continuous">
+    <parent link="bl_wheel_mount_link"/>
+    <child link="bl_wheel_link"/>
+    <origin xyz="0 0 -0.27" rpy="0 0 0"/>
+    <axis xyz="0 1 0"/>
+    <limit effort="100" velocity="10"/>
+  </joint>
+  <!-- ===================== BACK RIGHT WHEEL MOUNT ===================== -->
+  <link name="br_wheel_mount_link">
+    <inertial>
+      <origin xyz="0 0 0" rpy="0 0 0"/>
+      <mass value="0.162"/>
+      <inertia ixx="0.0002" iyy="0.00012" izz="0.00012" ixy="0" ixz="0" iyz="0"/>
+    </inertial>
+    <visual>
+      <origin xyz="0 0.06 -0.269" rpy="0 0 3.14159"/>
+      <geometry>
+        <mesh filename="package://indomitus_rover_description/meshes/suspension/wheel_mount.stl" scale="0.001 0.001 0.001"/>
+      </geometry>
+      <material name="orange_mount"/>
+    </visual>
+    <collision>
+      <origin xyz="0 -0.11125 -0.18" rpy="0 0 0"/>
+      <geometry>
+        <box size="0.07 0.0625 0.25"/>
+      </geometry>
+    </collision>
+  </link>
+  <joint name="br_wheel_mount_joint" type="revolute">
+    <parent link="r_rocker_link"/>
+    <child link="br_wheel_mount_link"/>
+    <origin xyz="-0.53 0 0" rpy="0 0 0"/>
+    <axis xyz="0 0 1"/>
+    <limit lower="-1.5708" upper="1.5708" effort="500" velocity="2"/>
+    <dynamics damping="0.5" friction="0.3"/>
+  </joint>
+  <!-- ===================== BACK RIGHT WHEEL ===================== -->
+  <link name="br_wheel_link">
+    <inertial>
+      <origin xyz="0 0 0" rpy="0 0 0"/>
+      <mass value="0.5"/>
+      <inertia ixx="0.00563" iyy="0.00563" izz="0.01125" ixy="0" ixz="0" iyz="0"/>
+    </inertial>
+    <visual>
+      <origin xyz="0 0.06 0" rpy="-1.5708 0 3.14159"/>
+      <geometry>
+        <mesh filename="package://indomitus_rover_description/meshes/suspension/wheel.stl" scale="0.001 0.001 0.001"/>
+      </geometry>
+      <material name="dark_wheel"/>
+    </visual>
+    <collision>
+      <origin xyz="0 0 0" rpy="-1.5708 0 0"/>
+      <geometry>
+        <cylinder radius="0.15" length="0.12"/>
+      </geometry>
+    </collision>
+  </link>
+  <joint name="br_wheel_joint" type="continuous">
+    <parent link="br_wheel_mount_link"/>
+    <child link="br_wheel_link"/>
+    <origin xyz="0 0 -0.27" rpy="0 0 0"/>
+    <axis xyz="0 1 0"/>
+    <limit effort="100" velocity="10"/>
+  </joint>
+</robot>
+<!-- <?xml version="1.0"?>
 <robot name="indomitus_s1" xmlns:xacro="https://www.ros.org/wiki/xacro">
   <xacro:arg name="name" default=""/>
@@ -21,3 +388,3 @@
   <xacro:wheel name="bl"  x="-0.53" y="0" z="0" side="1"  base_rocker="l" tf_prefix="${tf_prefix}"/>
   <xacro:wheel name="br" x="-0.53" y="0" z="0" side="-1" base_rocker="r" tf_prefix="${tf_prefix}"/>
-</robot>
+</robot> -->

File: src/indomitus_rover_sim/urdf/gazebo_plugins.urdf.xacro (robot description, xacro)
@@ -46,4 +46,14 @@
       <state_interface name="velocity"/>
     </joint>
+    <joint name="l_rocker_joint">
+      <!-- <command_interface name="position"/> -->
+      <state_interface name="position"/>
+      <state_interface name="velocity"/>
+    </joint>
+    <joint name="r_rocker_joint">
+      <command_interface name="position"/>
+      <state_interface name="position"/>
+      <state_interface name="velocity"/>
+    </joint>
   </ros2_control>
   <!-- gz_ros2_control plugin -->
