Commit message: Feature/suspension/3d model of suspension gazebo (#109)
* Rename packages names to new rover name indomitus_rover

* Raname bringup luanch files into rviz or robot_state_publisher

* Add RViz docs, move docker-compose to docker/, add startup warnings

* Adapt docs for ubuntu

* Fix docker-compose, localize ros2

* First working version; add gazebo launch files; add inertia to wheels; Add gazebo-ros2 topics bridge

* Fix wheel position

* Add rover_world.sdf; fix urdf model files; fix docs

* Add can_bridge node

* Fix bridge; fix docs for gazebo

* fix launch + add rover_world.sdf to spawn

* Add icr_controller_node

* add rgb camera sensor

* Fix control via teleop_twist

* Add docs for working version of simulation

* Add dependencies for rviz2; Add collisions for wheel_mount and rocker

* Temporary remove collision for rocker, FIX required, what is problem

* Add sdf files and scripts for gz with sdf; rename launch files

* Add working version of rover using sdf files

* Merge diff-bar branch to 3d-model branch

* Remove outdated docs

* Differential bar soft emulation with urdf model, working version

* Attached camera to camera_link in bridge_parameters

* Remove hardcoded world, add parameters to launch.py files

* Add header file for rocker_soft_mimic; replace humble with jazzy in docs

* refactor(launch): move config to yaml, decompose launch entry point

* Fix camera topic names, rqt output; fix license copyrights

* Try 2: Fix camera topic names, rqt output; fix license copyrights

---------

Co-authored-by: yaryna-zabchuk <yarunazabchuk@gmail.com>

File: src/indomitus_rover_description/urdf/indomitus_rover_s1.urdf.xacro (robot description, xacro)
@@ -1,21 +1,367 @@
 <?xml version="1.0"?>
-<robot name="indomitus_s1" xmlns:xacro="http://playerstage.sourceforge.net/gazebo/xmlschema/#xacro">
-  <xacro:arg name="name" default=""/>
-  <xacro:property name="_name" value="$(arg name)"/>
-  <xacro:if value="${_name != ''}">
-    <xacro:property name="tf_prefix" value="${_name}/"/>
-  </xacro:if>
-  <xacro:if value="${_name == ''}">
-    <xacro:property name="tf_prefix" value=""/>
-  </xacro:if>
-  <xacro:include filename="$(find indomitus_rover_description)/urdf/suspension.urdf.xacro"/>
-  <xacro:include filename="$(find indomitus_rover_description)/urdf/rocker.urdf.xacro"/>
-  <xacro:include filename="$(find indomitus_rover_description)/urdf/wheel.urdf.xacro"/>
-  <xacro:suspension xyz="0 0 0" tf_prefix="${tf_prefix}"/>
-  <xacro:rocker name="left"  xyz="0 0.305 0"  side="1"  base_axii="suspension_base_link" tf_prefix="${tf_prefix}"/>
-  <xacro:rocker name="right" xyz="0 -0.305 0" side="-1" base_axii="suspension_base_link" tf_prefix="${tf_prefix}"/>
-  <xacro:wheel name="front_left"  x="0.53" y="0" z="0" side="1" base_rocker="left" tf_prefix="${tf_prefix}"/>
-  <xacro:wheel name="front_right" x="0.53" y="0" z="0" side="-1" base_rocker="right" tf_prefix="${tf_prefix}"/>
-  <xacro:wheel name="back_left"  x="-0.53" y="0" z="0" side="1"  base_rocker="left" tf_prefix="${tf_prefix}"/>
-  <xacro:wheel name="back_right" x="-0.53" y="0" z="0" side="-1" base_rocker="right" tf_prefix="${tf_prefix}"/>
+<robot name="indomitus_s1" xmlns:xacro="http://www.ros.org/wiki/xacro">
+  <!-- ===================== MATERIALS ===================== -->
+  <material name="blue_body">
+    <color rgba="0.2 0.4 0.8 1"/>
+  </material>
+  <material name="grey_structure">
+    <color rgba="0.6 0.6 0.6 1"/>
+  </material>
+  <material name="orange_mount">
+    <color rgba="0.8 0.4 0.0 1"/>
+  </material>
+  <material name="dark_wheel">
+    <color rgba="0.1 0.1 0.1 1"/>
+  </material>
+  <material name="red_axii">
+    <color rgba="0.4 0.4 0.4 1"/>
+  </material>
+  <!-- ===================== BASE ===================== -->
+  <link name="base_link">
+    <inertial>
+      <mass value="0.1"/>
+      <inertia ixx="0.01" iyy="0.01" izz="0.01" ixy="0" ixz="0" iyz="0"/>
+    </inertial>
+  </link>
+  <!-- ===================== SUSPENSION BASE AXII ===================== -->
+  <link name="suspension_base_axii_link">
+    <inertial>
+      <origin xyz="0 0 0" rpy="0 0 0"/>
+      <mass value="0.5"/>
+      <inertia ixx="0.5" iyy="0.5" izz="1.0" ixy="0" ixz="0" iyz="0"/>
+    </inertial>
+    <visual>
+      <origin xyz="0 -0.325 0" rpy="0 0 0"/>
+      <geometry>
+        <mesh filename="package://indomitus_rover_description/meshes/suspension/central_axii.stl" scale="0.001 0.001 0.001"/>
+      </geometry>
+      <material name="red_axii"/>
+    </visual>
+    <collision>
+      <origin xyz="0 0 0" rpy="0 0 0"/>
+      <geometry>
+        <box size="0.1 0.65 0.05"/>
+      </geometry>
+    </collision>
+  </link>
+  <joint name="suspension_base_axii_joint" type="fixed">
+    <parent link="base_link"/>
+    <child link="suspension_base_axii_link"/>
+    <origin xyz="0 0 0" rpy="0 0 0"/>
+  </joint>
+  <!-- ===================== MAIN BODY ===================== -->
+  <link name="main_body_link">
+    <inertial>
+      <origin xyz="0 0 0" rpy="0 0 0"/>
+      <mass value="40.0"/>
+      <inertia ixx="0.608" iyy="1.283" izz="1.733" ixy="0" ixz="0" iyz="0"/>
+    </inertial>
+    <visual>
+      <origin xyz="0 0 0" rpy="0 0 0"/>
+      <geometry>
+        <box size="0.6 0.4 0.2"/>
+      </geometry>
+      <material name="blue_body"/>
+    </visual>
+    <collision>
+      <origin xyz="0 0 0" rpy="0 0 0"/>
+      <geometry>
+        <box size="0.6 0.4 0.15"/>
+      </geometry>
+    </collision>
+  </link>
+  <joint name="main_body_joint" type="fixed">
+    <parent link="suspension_base_axii_link"/>
+    <child link="main_body_link"/>
+    <origin xyz="-0.04 0 0.05" rpy="0 0 0"/>
+  </joint>
+  <!-- ===================== CAMERA ===================== -->
+  <xacro:include filename="$(find indomitus_rover_description)/urdf/camera.urdf.xacro"/>
+  <xacro:camera/>
+  <!-- ===================== LEFT ROCKER ===================== -->
+  <link name="l_rocker_link">
+    <inertial>
+      <origin xyz="0 0 0" rpy="0 0 0"/>
+      <mass value="1.0"/>
+      <inertia ixx="0.01" iyy="0.01" izz="0.01" ixy="0" ixz="0" iyz="0"/>
+    </inertial>
+    <visual>
+      <origin xyz="-0.55 0.02 -0.04" rpy="0 0 0"/>
+      <geometry>
+        <mesh filename="package://indomitus_rover_description/meshes/suspension/rocker.stl" scale="0.001 0.001 0.001"/>
+      </geometry>
+      <material name="grey_structure"/>
+    </visual>
+    <collision>
+      <origin xyz="0 0 0" rpy="0 0 0"/>
+      <geometry>
+        <box size="1.1 0.04 0.08"/>
+      </geometry>
+    </collision>
+  </link>
+  <joint name="l_rocker_joint" type="revolute">
+    <parent link="suspension_base_axii_link"/>
+    <child link="l_rocker_link"/>
+    <origin xyz="0 0.305 0" rpy="0 0 0"/>
+    <axis xyz="0 1 0"/>
+    <limit lower="-0.5" upper="0.5" effort="100" velocity="1.0"/>
+    <dynamics damping="0.5" friction="0.1"/>
+  </joint>
+  <!-- ===================== RIGHT ROCKER ===================== -->
+  <link name="r_rocker_link">
+    <inertial>
+      <origin xyz="0 0 0" rpy="0 0 0"/>
+      <mass value="1.0"/>
+      <inertia ixx="0.01" iyy="0.01" izz="0.01" ixy="0" ixz="0" iyz="0"/>
+    </inertial>
+    <visual>
+      <origin xyz="-0.55 0.02 -0.04" rpy="0 0 0"/>
+      <geometry>
+        <mesh filename="package://indomitus_rover_description/meshes/suspension/rocker.stl" scale="0.001 0.001 0.001"/>
+      </geometry>
+      <material name="grey_structure"/>
+    </visual>
+    <collision>
+      <origin xyz="0 0 0" rpy="0 0 0"/>
+      <geometry>
+        <box size="1.1 0.04 0.08"/>
+      </geometry>
+    </collision>
+  </link>
+  <joint name="r_rocker_joint" type="revolute">
+    <parent link="suspension_base_axii_link"/>
+    <child link="r_rocker_link"/>
+    <origin xyz="0 -0.305 0" rpy="0 0 0"/>
+    <axis xyz="0 1 0"/>
+    <limit lower="-0.5" upper="0.5" effort="100" velocity="1.0"/>
+    <dynamics damping="0.5" friction="0.1"/>
+  </joint>
+  <!-- ===================== FRONT LEFT WHEEL MOUNT ===================== -->
+  <link name="fl_wheel_mount_link">
+    <inertial>
+      <origin xyz="0 0 0" rpy="0 0 0"/>
+      <mass value="0.162"/>
+      <inertia ixx="0.0002" iyy="0.00012" izz="0.00012" ixy="0" ixz="0" iyz="0"/>
+    </inertial>
+    <visual>
+      <origin xyz="0 -0.06 -0.269" rpy="0 0 0"/>
+      <geometry>
+        <mesh filename="package://indomitus_rover_description/meshes/suspension/wheel_mount.stl" scale="0.001 0.001 0.001"/>
+      </geometry>
+      <material name="orange_mount"/>
+    </visual>
+    <collision>
+      <origin xyz="0 0.11125 -0.18" rpy="0 0 0"/>
+      <geometry>
+        <box size="0.07 0.0625 0.25"/>
+      </geometry>
+    </collision>
+  </link>
+  <joint name="fl_wheel_mount_joint" type="revolute">
+    <parent link="l_rocker_link"/>
+    <child link="fl_wheel_mount_link"/>
+    <origin xyz="0.53 0 0" rpy="0 0 0"/>
+    <axis xyz="0 0 1"/>
+    <limit lower="-1.5708" upper="1.5708" effort="500" velocity="2"/>
+    <dynamics damping="0.5" friction="0.3"/>
+  </joint>
+  <!-- ===================== FRONT LEFT WHEEL ===================== -->
+  <link name="fl_wheel_link">
+    <inertial>
+      <origin xyz="0 0 0" rpy="0 0 0"/>
+      <mass value="0.5"/>
+      <inertia ixx="0.00563" iyy="0.00563" izz="0.01125" ixy="0" ixz="0" iyz="0"/>
+    </inertial>
+    <visual>
+      <origin xyz="0 -0.06 0" rpy="-1.5708 0 0"/>
+      <geometry>
+        <mesh filename="package://indomitus_rover_description/meshes/suspension/wheel.stl" scale="0.001 0.001 0.001"/>
+      </geometry>
+      <material name="dark_wheel"/>
+    </visual>
+    <collision>
+      <origin xyz="0 0 0" rpy="1.5708 0 0"/>
+      <geometry>
+        <cylinder radius="0.15" length="0.12"/>
+      </geometry>
+    </collision>
+  </link>
+  <joint name="fl_wheel_joint" type="continuous">
+    <parent link="fl_wheel_mount_link"/>
+    <child link="fl_wheel_link"/>
+    <origin xyz="0 0 -0.27" rpy="0 0 0"/>
+    <axis xyz="0 1 0"/>
+    <limit effort="100" velocity="10"/>
+  </joint>
+  <!-- ===================== FRONT RIGHT WHEEL MOUNT ===================== -->
+  <link name="fr_wheel_mount_link">
+    <inertial>
+      <origin xyz="0 0 0" rpy="0 0 0"/>
+      <mass value="0.162"/>
+      <inertia ixx="0.0002" iyy="0.00012" izz="0.00012" ixy="0" ixz="0" iyz="0"/>
+    </inertial>
+    <visual>
+      <origin xyz="0 0.06 -0.269" rpy="0 0 3.14159"/>
+      <geometry>
+        <mesh filename="package://indomitus_rover_description/meshes/suspension/wheel_mount.stl" scale="0.001 0.001 0.001"/>
+      </geometry>
+      <material name="orange_mount"/>
+    </visual>
+    <collision>
+      <origin xyz="0 -0.11125 -0.18" rpy="0 0 0"/>
+      <geometry>
+        <box size="0.07 0.0625 0.25"/>
+      </geometry>
+    </collision>
+  </link>
+  <joint name="fr_wheel_mount_joint" type="revolute">
+    <parent link="r_rocker_link"/>
+    <child link="fr_wheel_mount_link"/>
+    <origin xyz="0.53 0 0" rpy="0 0 0"/>
+    <axis xyz="0 0 1"/>
+    <limit lower="-1.5708" upper="1.5708" effort="500" velocity="2"/>
+    <dynamics damping="0.5" friction="0.3"/>
+  </joint>
+  <!-- ===================== FRONT RIGHT WHEEL ===================== -->
+  <link name="fr_wheel_link">
+    <inertial>
+      <origin xyz="0 0 0" rpy="0 0 0"/>
+      <mass value="0.5"/>
+      <inertia ixx="0.00563" iyy="0.00563" izz="0.01125" ixy="0" ixz="0" iyz="0"/>
+    </inertial>
+    <visual>
+      <origin xyz="0 0.06 0" rpy="-1.5708 0 3.14159"/>
+      <geometry>
+        <mesh filename="package://indomitus_rover_description/meshes/suspension/wheel.stl" scale="0.001 0.001 0.001"/>
+      </geometry>
+      <material name="dark_wheel"/>
+    </visual>
+    <collision>
+      <origin xyz="0 0 0" rpy="-1.5708 0 0"/>
+      <geometry>
+        <cylinder radius="0.15" length="0.12"/>
+      </geometry>
+    </collision>
+  </link>
+  <joint name="fr_wheel_joint" type="continuous">
+    <parent link="fr_wheel_mount_link"/>
+    <child link="fr_wheel_link"/>
+    <origin xyz="0 0 -0.27" rpy="0 0 0"/>
+    <axis xyz="0 1 0"/>
+    <limit effort="100" velocity="10"/>
+  </joint>
+  <!-- ===================== BACK LEFT WHEEL MOUNT ===================== -->
+  <link name="bl_wheel_mount_link">
+    <inertial>
+      <origin xyz="0 0 0" rpy="0 0 0"/>
+      <mass value="0.162"/>
+      <inertia ixx="0.0002" iyy="0.00012" izz="0.00012" ixy="0" ixz="0" iyz="0"/>
+    </inertial>
+    <visual>
+      <origin xyz="0 -0.06 -0.269" rpy="0 0 0"/>
+      <geometry>
+        <mesh filename="package://indomitus_rover_description/meshes/suspension/wheel_mount.stl" scale="0.001 0.001 0.001"/>
+      </geometry>
+      <material name="orange_mount"/>
+    </visual>
+    <collision>
+      <origin xyz="0 0.11125 -0.18" rpy="0 0 0"/>
+      <geometry>
+        <box size="0.07 0.0625 0.25"/>
+      </geometry>
+    </collision>
+  </link>
+  <joint name="bl_wheel_mount_joint" type="revolute">
+    <parent link="l_rocker_link"/>
+    <child link="bl_wheel_mount_link"/>
+    <origin xyz="-0.53 0 0" rpy="0 0 0"/>
+    <axis xyz="0 0 1"/>
+    <limit lower="-1.5708" upper="1.5708" effort="500" velocity="2"/>
+    <dynamics damping="0.5" friction="0.3"/>
+  </joint>
+  <!-- ===================== BACK LEFT WHEEL ===================== -->
+  <link name="bl_wheel_link">
+    <inertial>
+      <origin xyz="0 0 0" rpy="0 0 0"/>
+      <mass value="0.5"/>
+      <inertia ixx="0.00563" iyy="0.00563" izz="0.01125" ixy="0" ixz="0" iyz="0"/>
+    </inertial>
+    <visual>
+      <origin xyz="0 -0.06 0" rpy="-1.5708 0 0"/>
+      <geometry>
+        <mesh filename="package://indomitus_rover_description/meshes/suspension/wheel.stl" scale="0.001 0.001 0.001"/>
+      </geometry>
+      <material name="dark_wheel"/>
+    </visual>
+    <collision>
+      <origin xyz="0 0 0" rpy="1.5708 0 0"/>
+      <geometry>
+        <cylinder radius="0.15" length="0.12"/>
+      </geometry>
+    </collision>
+  </link>
+  <joint name="bl_wheel_joint" type="continuous">
+    <parent link="bl_wheel_mount_link"/>
+    <child link="bl_wheel_link"/>
+    <origin xyz="0 0 -0.27" rpy="0 0 0"/>
+    <axis xyz="0 1 0"/>
+    <limit effort="100" velocity="10"/>
+  </joint>
+  <!-- ===================== BACK RIGHT WHEEL MOUNT ===================== -->
+  <link name="br_wheel_mount_link">
+    <inertial>
+      <origin xyz="0 0 0" rpy="0 0 0"/>
+      <mass value="0.162"/>
+      <inertia ixx="0.0002" iyy="0.00012" izz="0.00012" ixy="0" ixz="0" iyz="0"/>
+    </inertial>
+    <visual>
+      <origin xyz="0 0.06 -0.269" rpy="0 0 3.14159"/>
+      <geometry>
+        <mesh filename="package://indomitus_rover_description/meshes/suspension/wheel_mount.stl" scale="0.001 0.001 0.001"/>
+      </geometry>
+      <material name="orange_mount"/>
+    </visual>
+    <collision>
+      <origin xyz="0 -0.11125 -0.18" rpy="0 0 0"/>
+      <geometry>
+        <box size="0.07 0.0625 0.25"/>
+      </geometry>
+    </collision>
+  </link>
+  <joint name="br_wheel_mount_joint" type="revolute">
+    <parent link="r_rocker_link"/>
+    <child link="br_wheel_mount_link"/>
+    <origin xyz="-0.53 0 0" rpy="0 0 0"/>
+    <axis xyz="0 0 1"/>
+    <limit lower="-1.5708" upper="1.5708" effort="500" velocity="2"/>
+    <dynamics damping="0.5" friction="0.3"/>
+  </joint>
+  <!-- ===================== BACK RIGHT WHEEL ===================== -->
+  <link name="br_wheel_link">
+    <inertial>
+      <origin xyz="0 0 0" rpy="0 0 0"/>
+      <mass value="0.5"/>
+      <inertia ixx="0.00563" iyy="0.00563" izz="0.01125" ixy="0" ixz="0" iyz="0"/>
+    </inertial>
+    <visual>
+      <origin xyz="0 0.06 0" rpy="-1.5708 0 3.14159"/>
+      <geometry>
+        <mesh filename="package://indomitus_rover_description/meshes/suspension/wheel.stl" scale="0.001 0.001 0.001"/>
+      </geometry>
+      <material name="dark_wheel"/>
+    </visual>
+    <collision>
+      <origin xyz="0 0 0" rpy="-1.5708 0 0"/>
+      <geometry>
+        <cylinder radius="0.15" length="0.12"/>
+      </geometry>
+    </collision>
+  </link>
+  <joint name="br_wheel_joint" type="continuous">
+    <parent link="br_wheel_mount_link"/>
+    <child link="br_wheel_link"/>
+    <origin xyz="0 0 -0.27" rpy="0 0 0"/>
+    <axis xyz="0 1 0"/>
+    <limit effort="100" velocity="10"/>
+  </joint>
 </robot>
